Commit message: Register gantry joints in ros2_control so their TF is published
The 3 new gantry joints were in no ros2_control block, so joint_state_broadcaster
never published their positions; robot_state_publisher then couldn't place the
links and RViz drew them at the world origin (white, on the floor).

- robodrill_diffdrive_control.xacro: add a gantry_controller ros2_control system
  (GazeboSimSystem in sim, mock otherwise) exposing position/velocity for
  gantry_y/x/rot joints.
- diffdrive_controllers.yaml: add the 3 joints to joint_state_broadcaster and add
  a gantry_position_controller for commanding/holding them.

File: robo_drill_description/description/robodrill_diffdrive_control.xacro (robot description, xacro)
@@ -79,4 +79,37 @@
         </joint>
     </ros2_control>
+    <!-- Gantry - Stage 2 (Y), Stage 3 (X) and end rotation.
+         Registered so the joint_state_broadcaster publishes their positions
+         (otherwise robot_state_publisher can't place these links and RViz
+         shows them at the world origin). Real gantry hardware is not yet
+         implemented, so non-simulation uses a mock system for now. -->
+    <ros2_control name="gantry_controller" type="system">
+        <xacro:if value="$(arg simulation)">
+            <hardware>
+                <plugin>gz_ros2_control/GazeboSimSystem</plugin>
+            </hardware>
+        </xacro:if>
+        <xacro:unless value="$(arg simulation)">
+            <hardware>
+                <plugin>mock_components/GenericSystem</plugin>
+                <param name="calculate_dynamics">true</param>
+            </hardware>
+        </xacro:unless>
+        <joint name="gantry_y_joint">
+            <command_interface name="position"/>
+            <state_interface name="position"/>
+            <state_interface name="velocity"/>
+        </joint>
+        <joint name="gantry_x_joint">
+            <command_interface name="position"/>
+            <state_interface name="position"/>
+            <state_interface name="velocity"/>
+        </joint>
+        <joint name="gantry_rot_joint">
+            <command_interface name="position"/>
+            <state_interface name="position"/>
+            <state_interface name="velocity"/>
+        </joint>
+    </ros2_control>
     <xacro:if value="$(arg simulation)">
         <xacro:if value="$(arg base_only)">
