Commit message: Replace column+UR10e with 3-stage linear gantry (Z/Y/X) + end rotation
- pokeye_base.urdf: keep column_link as Stage 1 (Z lift); add gantry_y (Y side),
  gantry_x (X reach) prismatic stages and gantry_rot revolute end, all as boxes;
  gravity disabled so they hold pose in Gazebo (geometry placeholders).
- mobile_manipulator.urdf.xacro: remove UR10e + sensor_plate mount.

File: robo_drill_description/description/mobile_manipulator.urdf.xacro (robot description, xacro)
@@ -114,56 +114,8 @@
         origin_rpy="-0.143 1.541 -0.145"
     />
-    <xacro:include filename="$(find arm_control)/urdf/ur_macro.xacro"/>
-    <!-- Mount UR10e arm on column_link -->
-    <xacro:ur_robot
-        name="$(arg ur_type)"
-        tf_prefix="$(arg tf_prefix)"
-        parent="column_link"
-        joint_limits_parameters_file="$(arg joint_limit_params)"
-        kinematics_parameters_file="$(arg kinematics_params)"
-        physical_parameters_file="$(arg physical_params)"
-        visual_parameters_file="$(arg visual_params)"
-        transmission_hw_interface="$(arg transmission_hw_interface)"
-        safety_limits="$(arg safety_limits)"
-        safety_pos_margin="$(arg safety_pos_margin)"
-        safety_k_position="$(arg safety_k_position)"
-        use_fake_hardware="$(arg use_fake_hardware)"
-        fake_sensor_commands="$(arg fake_sensor_commands)"
-        sim_gazebo="$(arg sim_gazebo)"
-        sim_ignition="$(arg sim_ignition)"
-        headless_mode="$(arg headless_mode)"
-        initial_positions="${xacro.load_yaml(initial_positions_file)}"
-        use_tool_communication="$(arg use_tool_communication)"
-        tool_voltage="$(arg tool_voltage)"
-        tool_parity="$(arg tool_parity)"
-        tool_baud_rate="$(arg tool_baud_rate)"
-        tool_stop_bits="$(arg tool_stop_bits)"
-        tool_rx_idle_chars="$(arg tool_rx_idle_chars)"
-        tool_tx_idle_chars="$(arg tool_tx_idle_chars)"
-        tool_device_name="$(arg tool_device_name)"
-        tool_tcp_port="$(arg tool_tcp_port)"
-        robot_ip="$(arg robot_ip)"
-        script_filename="$(arg script_filename)"
-        output_recipe_filename="$(arg output_recipe_filename)"
-        input_recipe_filename="$(arg input_recipe_filename)"
-        reverse_ip="$(arg reverse_ip)"
-        script_command_port="$(arg script_command_port)"
-        reverse_port="$(arg reverse_port)"
-        script_sender_port="$(arg script_sender_port)"
-        trajectory_port="$(arg trajectory_port)"
-        arm_dyn_scale="$(arg arm_dyn_scale)"
-        ee_cylinder_length="$(arg ee_cylinder_length)"
-        ee_cylinder_radius="$(arg ee_cylinder_radius)"
-        sensors_offset="$(arg sensors_offset)"
-    >
-        <!--! Arm mounting position  of arm_base_link relative to column_link -->
-        <origin xyz="0.0 0.0 0.73"
-                rpy="0.0 0.0 -2.3562"/>
-    </xacro:ur_robot>
-    <xacro:include filename="$(find arm_control)/urdf/sensor_plate.urdf.xacro"/>
-    <xacro:sensor_plate
-     parent_link="$(arg tf_prefix)ee_cylinder_link"
-     tf_prefix="$(arg tf_prefix)"
-     ee_cylinder_length="$(arg ee_cylinder_length)"/>
+    <!-- Pokeye has no UR10e manipulator. The 3-stage linear-actuator gantry
+         (column_link -> gantry_y_link -> gantry_x_link -> gantry_rot_link) is
+         defined in pokeye_base.urdf and is shared by both robo_drill.urdf.xacro
+         and this file. The former UR10e + sensor_plate mount has been removed. -->
     <xacro:if value="$(arg sim_ignition)">
         <gazebo>

File: robo_drill_description/description/pokeye_base.urdf (robot description, URDF)
Before this commit: robot Pokeye, 10 links, 9 joints
Links:
- added link gantry_rot_link, mass 1.0; collision box size=0.08 0.08 0.15; visual box size=0.08 0.08 0.15
- added link gantry_x_link, mass 2.0; collision box size=0.50 0.10 0.10; visual box size=0.50 0.10 0.10
- added link gantry_y_link, mass 3.0; collision box size=0.12 0.50 0.10; visual box size=0.12 0.50 0.10
Joints:
- added joint gantry_rot_joint: type revolute, parent gantry_x_link, child gantry_rot_link, origin xyz=0.40 0 0.05 rpy=0 0 0, axis 0 0 1, limit lower=-3.1416 upper=3.1416 effort=100.0 velocity=1.0
- added joint gantry_x_joint: type prismatic, parent gantry_y_link, child gantry_x_link, origin xyz=0 0 0.10 rpy=0 0 0, axis 1 0 0, limit lower=0.0 upper=0.40 effort=500.0 velocity=0.2
- added joint gantry_y_joint: type prismatic, parent column_link, child gantry_y_link, origin xyz=0 0 0.73 rpy=0 0 0, axis 0 1 0, limit lower=-0.25 upper=0.25 effort=500.0 velocity=0.2

Commit message: Refactor column into gantry Z-stage; add Z to UI; strip self.arm_* refs
- Renamed column_link/column_joint -> gantry_z_link/gantry_z_joint (Stage 1,
  vertical Z lift, 0-0.9 m).
- Folded gantry_z into the single gantry_position_controller (removed the
  separate column_controller/column_position_controller ros2_control system and
  their controller configs); joint order is now [Z, Y, X, rot].
- Updated joint_state_broadcaster, sim.launch.py and robot.launch.py spawners
  (column_* spawners -> gantry_position_controller); updated column_link frame
  references in hybrid_simulation.launch.py and mobile_manipulator comment.
- UI Gantry Control tab now has a Z-lift slider (order Z,Y,X,rot) and publishes
  the 4-value command; updated tooltip/log and UI_GUIDE.
- Stripped all remaining self.arm_* references from the UI.

Note: python_nodes/goal_router.py still has column_* parameter defaults; it is a
standalone task-planner node (not launched by the platform) and was left as-is.

File: robo_drill_description/description/mobile_manipulator.urdf.xacro (robot description, xacro)
@@ -115,5 +115,5 @@
     />
     <!-- Pokeye has no UR10e manipulator. The 3-stage linear-actuator gantry
-         (column_link -> gantry_y_link -> gantry_x_link -> gantry_rot_link) is
+         (gantry_z_link -> gantry_y_link -> gantry_x_link -> gantry_rot_link) is
          defined in pokeye_base.urdf and is shared by both robo_drill.urdf.xacro
          and this file. The former UR10e + sensor_plate mount has been removed. -->

File: robo_drill_description/description/pokeye_base.urdf (robot description, URDF)
Before this commit: robot Pokeye, 13 links, 12 joints
Links:
- removed link column_link
- added link gantry_z_link, mass 1.0; collision box size=0.10 0.12 0.73; visual box size=0.10 0.12 0.73
Joints:
- removed joint column_joint
- added joint gantry_z_joint: type prismatic, parent turret_link, child gantry_z_link, origin xyz=0.2905 0 0 rpy=0 0 0, axis 0 0 1, limit lower=0.0 upper=0.9 effort=1000.0 velocity=0.1
- joint gantry_y_joint: parent column_link -> gantry_z_link

File: robo_drill_description/description/robodrill_diffdrive_control.xacro (robot description, xacro)
@@ -47,41 +47,10 @@
         </joint>
     </ros2_control>
-    <!-- Column Hardware Interface -->
-    <ros2_control name="column_controller" type="system">
-        <xacro:unless value="$(arg simulation)">
-            <xacro:unless value="$(arg use_mock_hardware)">
-                <hardware>
-                    <plugin>column_hw_interface/ColumnHardwareInterface</plugin>
-                    <param name="column_name">column_joint</param>
-                </hardware>
-            </xacro:unless>
-            <xacro:if value="$(arg use_mock_hardware)">
-                <hardware>
-                    <plugin>mock_components/GenericSystem</plugin>
-                    <param name="calculate_dynamics">true</param>
-                </hardware>
-            </xacro:if>
-        </xacro:unless>
-        <xacro:if value="$(arg simulation)">
-            <hardware>
-                <plugin>gz_ros2_control/GazeboSimSystem</plugin>
-            </hardware>
-        </xacro:if>
-        <joint name="column_joint">
-            <xacro:if value="$(arg simulation)">
-                <command_interface name="effort"/>
-            </xacro:if>
-            <xacro:unless value="$(arg simulation)">
-                <command_interface name="position"/>
-            </xacro:unless>
-            <state_interface name="position"/>
-            <state_interface name="velocity"/>
-        </joint>
-    </ros2_control>
-    <!-- Gantry - Stage 2 (Y), Stage 3 (X) and end rotation.
-         Registered so the joint_state_broadcaster publishes their positions
-         (otherwise robot_state_publisher can't place these links and RViz
-         shows them at the world origin). Real gantry hardware is not yet
-         implemented, so non-simulation uses a mock system for now. -->
+    <!-- Gantry - Stage 1 (Z lift), Stage 2 (Y), Stage 3 (X) and end rotation.
+         All four stages are one linear-actuator gantry driven by a single
+         gantry_position_controller. Registered here so the joint_state_broadcaster
+         publishes their positions (otherwise robot_state_publisher can't place
+         these links and RViz shows them at the world origin). Real gantry hardware
+         is not yet implemented, so non-simulation uses a mock system for now. -->
     <ros2_control name="gantry_controller" type="system">
         <xacro:if value="$(arg simulation)">
@@ -96,4 +65,9 @@
             </hardware>
         </xacro:unless>
+        <joint name="gantry_z_joint">
+            <command_interface name="position"/>
+            <state_interface name="position"/>
+            <state_interface name="velocity"/>
+        </joint>
         <joint name="gantry_y_joint">
             <command_interface name="position"/>

Commit message: Refactor mobile manipulator configuration and UI updates
- Updated joint names in diffdrive_controllers.yaml to reflect new gantry joint structure.
- Removed obsolete column controller configurations in mobile_manipulator_controllers.yaml.
- Adjusted gantry joint parameters in mobile_manipulator_controllers.yaml.
- Modified navigation parameters in nav2_params_omni.yaml for improved path following.
- Updated UI_GUIDE.md to reflect changes in gantry control commands and joint names.
- Changed manipulator.launch.py to load the correct parameters file for the mobile manipulator.
- Disabled dynamic footprint publisher in navigation_launch.py for better performance.
- Updated URDF/XACRO files for the mobile manipulator to reflect new joint names and configurations.
- Adjusted mass and inertia properties in pokeye_base.urdf for better simulation accuracy.
- Updated UI.py to reflect new gantry joint names and improved control panel layout.

File: robo_drill_description/description/mobile_manipulator.urdf.xacro (robot description, xacro)
@@ -67,21 +67,21 @@
     <!-- Front-right Sick lidar -->
     <xacro:sick_multiscan_sensor
-        parent_link="os_sensor_mount"
+        parent_link="turret_link"
         namespace="front"
         sick_link="front_sick_scan"
         sick_scan_link="front_sick"
         sick_imu_link="front_sick_imu"
-        origin_xyz="-0.002 0.243 -0.081"
-        origin_rpy="1.130 0.938 1.453"
+        origin_xyz="0.38 -0.35 0.08"
+        origin_rpy="0.0 0.0 0.0"
     />
     <!-- Sick lidar at back-left of robot -->
     <xacro:sick_multiscan_sensor
-        parent_link="os_sensor_mount"
+        parent_link="turret_link"
         namespace="rear"
         sick_link="rear_sick_scan"
         sick_scan_link="rear_sick"
         sick_imu_link="rear_sick_imu"
-        origin_xyz="-0.002 -0.252 -0.788"
-        origin_rpy="-1.98 -0.973 -1.496"
+        origin_xyz="-0.42 0.35 0.08"
+        origin_rpy="0.0 0.0 0.0"
     />
     <!-- Add third sick lidar only in simulation -->
@@ -115,5 +115,5 @@
     />
     <!-- Pokeye has no UR10e manipulator. The 3-stage linear-actuator gantry
-         (gantry_z_link -> gantry_y_link -> gantry_x_link -> gantry_rot_link) is
+         (gantry_lift1_link -> gantry_lift2_link -> gantry_lateral_link -> gantry_rotate_link) is
          defined in pokeye_base.urdf and is shared by both robo_drill.urdf.xacro
          and this file. The former UR10e + sensor_plate mount has been removed. -->

File: robo_drill_description/description/pokeye_base.urdf (robot description, URDF)
Before this commit: robot Pokeye, 13 links, 12 joints
Links:
- removed link gantry_rot_link
- removed link gantry_x_link
- removed link gantry_y_link
- removed link gantry_z_link
- added link drill_tip
- added link gantry_lateral_link, mass 1.0; collision mesh filename=package://robo_drill/robo_drill_description/meshes/rotatory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 scale=0.001 0.001 0.001; visual mesh filename=package://robo_drill/robo_drill_description/meshes/rotatory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 scale=0.001 0.001 0.001
- added link gantry_lift1_link, mass 0.5; collision mesh filename=package://robo_drill/robo_drill_description/meshes/d_e_stag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 scale=0.001 0.001 0.001; visual mesh filename=package://robo_drill/robo_drill_description/meshes/d_e_stag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 scale=0.001 0.001 0.001
- added link gantry_lift2_link, mass 1.5; collision mesh filename=package://robo_drill/robo_drill_description/meshes/d_e_stag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 scale=0.001 0.001 0.001; visual mesh filename=package://robo_drill/robo_drill_description/meshes/d_e_stag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 scale=0.001 0.001 0.001
- added link gantry_rotate_link, mass 0.5; collision box size=0.08 0.08 0.15
- link base_link: mass 30.0 -> 15.0; geometry collision mesh filename=package://robo_drill/robo_drill_description/meshes/d_base_v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 scale=0.001 0.001 0.001; visual mesh filename=package://robo_drill/robo_drill_description/meshes/d_base_v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 scale=0.001 0.001 0.001
- link drivewhl_l_joint_link: mass 54.4811070994725 -> 27.24055354973625
- link drivewhl_r_joint_link: mass 54.4811070994725 -> 27.24055354973625
- link turret_caster_bl: mass 0.05 -> 0.025
- link turret_caster_br: mass 0.05 -> 0.025
- link turret_caster_fl: mass 0.05 -> 0.025
- link turret_caster_fr: mass 0.05 -> 0.025
- link turret_link: geometry collision mesh filename=package://robo_drill/robo_drill_description/meshes/d_e_stag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 scale=0.001 0.001 0.001; visual mesh filename=package://robo_drill/robo_drill_description/meshes/d_e_stag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 scale=0.001 0.001 0.001
Joints:
- removed joint gantry_rot_joint
- removed joint gantry_x_joint
- removed joint gantry_y_joint
- removed joint gantry_z_joint
- added joint drill_tip_joint: type fixed, parent gantry_rotate_link, child drill_tip, origin xyz=${drill_tip_x} ${drill_tip_y} ${drill_tip_z} rpy=${drill_tip_roll} ${drill_tip_pitch} ${drill_tip_yaw}
- added joint gantry_lateral_joint: type prismatic, parent gantry_lift2_link, child gantry_lateral_link, origin xyz=0 0 0.10 rpy=0 0 0, axis 0 1 0, limit lower=-0.196 upper=0.196 effort=500.0 velocity=0.2
- added joint gantry_lift1_joint: type prismatic, parent turret_link, child gantry_lift1_link, origin xyz=0.2905 0 0 rpy=0 0 0, axis 0 0 1, limit lower=-0.47 upper=0.40 effort=1000.0 velocity=0.1
- added joint gantry_lift2_joint: type prismatic, parent gantry_lift1_link, child gantry_lift2_link, origin xyz=0.19 0 0.423 rpy=0 0 0, axis 0 0 1, limit lower=0.0 upper=1.0 effort=500.0 velocity=0.2
- added joint gantry_rotate_joint: type revolute, parent gantry_lateral_link, child gantry_rotate_link, origin xyz=0.06 0.06 0.0 rpy=1.5708 0 1.5708, axis 0 0 1, limit lower=-3.1416 upper=3.1416 effort=100.0 velocity=1.0
- joint drivewhl_l_joint: origin xyz=0 0.18275 0 rpy=-1.5708 0 0 -> xyz=0 0.40275 0 rpy=-1.5708 0 0
- joint drivewhl_r_joint: origin xyz=0 -0.18275 0 rpy=-1.5708 0 0 -> xyz=0 -0.40275 0 rpy=-1.5708 0 0
- joint turret_joint: origin xyz=0.167 0 0.2575 rpy=0 0 0 -> xyz=0.40 0 0.2575 rpy=0 0 0
