Commit message: Refactor lidar and gantry configurations: update frame references, remove dome lidar, and adjust joint names in URDF and UI files.

File: robo_drill_description/description/mobile_manipulator.urdf.xacro (robot description, xacro)
@@ -63,5 +63,4 @@
     <xacro:include filename="pokeye_base.urdf"/>
     <xacro:include filename="sick_multiscan.xacro"/>
-    <xacro:include filename="os-dome.xacro"/>
     <xacro:include filename="realsense_camera.xacro"/>
     <!-- Front-right Sick lidar -->
@@ -85,35 +84,25 @@
         origin_rpy="0.0 0.0 0.0"
     />
-    <!-- Add third sick lidar only in simulation -->
-    <xacro:if value="$(arg simulation)">
-        <xacro:sick_multiscan_sensor
-            parent_link="os_sensor_mount"
-            namespace="dome"
-            sick_link="os_lidar"
-            sick_scan_link="dome_scan"
-            sick_imu_link="dome_imu"
-            origin_xyz="0 0 0"
-            origin_rpy="0 0 0"
-        />
-    </xacro:if>
     <!-- Front RealSense D435i (forward facing) - legacy frames/topics preserved -->
+    <!-- Parented directly to turret_link; origin composed from the previous
+         mount pose so the physical camera placement is unchanged. -->
     <xacro:realsense_d435
-        parent_link="os_sensor_mount"
+        parent_link="turret_link"
         camera_name="camera"
         topic_ns="camera/camera"
-        origin_xyz="0.0075 -0.128 0.015"
-        origin_rpy="-2.998 -1.541 -0.145"
+        origin_xyz="0.4495 0.1280 0.4600"
+        origin_rpy="-0.0015 -0.0295 0.0043"
     />
     <!-- Rear RealSense D435i (back of turret, for localization and mapping) -->
-    <!-- TODO: replace origin with the measured pose of the rear camera on os_sensor_mount -->
+    <!-- TODO: replace origin with the measured pose of the rear camera on turret_link -->
     <xacro:realsense_d435
-        parent_link="os_sensor_mount"
+        parent_link="turret_link"
         camera_name="camera_rear"
         topic_ns="camera_rear"
-        origin_xyz="0.0075 0.128 -0.84"
-        origin_rpy="-0.143 1.541 -0.145"
+        origin_xyz="-0.4055 -0.1280 0.4600"
+        origin_rpy="0.0021 -0.0295 3.1373"
     />
     <!-- Pokeye has no UR10e manipulator. The 3-stage linear-actuator gantry
-         (gantry_lift1_link -> gantry_lift2_link -> gantry_lateral_link -> gantry_rotate_link) is
+         (stage1_lift_link -> stage2_lift_link -> stage3_horizontal_link -> stage4_rotate_link) is
          defined in pokeye_base.urdf and is shared by both robo_drill.urdf.xacro
          and this file. The former UR10e + sensor_plate mount has been removed. -->

File: robo_drill_description/description/pokeye_base.urdf (robot description, URDF)
Before this commit: robot Pokeye, 14 links, 13 joints
Links:
- removed link gantry_lateral_link
- removed link gantry_lift1_link
- removed link gantry_lift2_link
- removed link gantry_rotate_link
- removed link turret_caster_bl
- removed link turret_caster_br
- removed link turret_caster_fl
- removed link turret_caster_fr
- added link stage1_lift_link, mass 0.5; collision mesh filename=package://robo_drill/robo_drill_description/meshes/d_e_stag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 scale=0.001 0.001 0.001; visual mesh filename=package://robo_drill/robo_drill_description/meshes/d_e_stag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 scale=0.001 0.001 0.001
- added link stage2_lift_link, mass 1.5; collision mesh filename=package://robo_drill/robo_drill_description/meshes/d_e_stag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 scale=0.001 0.001 0.001; visual mesh filename=package://robo_drill/robo_drill_description/meshes/d_e_stag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 scale=0.001 0.001 0.001
- added link stage3_horizontal_link, mass 1.0; collision mesh filename=package://robo_drill/robo_drill_description/meshes/rotatory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 scale=0.001 0.001 0.001; visual mesh filename=package://robo_drill/robo_drill_description/meshes/rotatory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 scale=0.001 0.001 0.001
- added link stage4_rotate_link, mass 0.5; collision box size=0.08 0.08 0.15
Joints:
- removed joint gantry_lateral_joint
- removed joint gantry_lift1_joint
- removed joint gantry_lift2_joint
- removed joint gantry_rotate_joint
- removed joint turret_caster_bl_joint
- removed joint turret_caster_br_joint
- removed joint turret_caster_fl_joint
- removed joint turret_caster_fr_joint
- added joint stage1_lift_joint: type prismatic, parent turret_link, child stage1_lift_link, origin xyz=0.2905 0 0 rpy=0 0 0, axis 0 0 1, limit lower=-0.47 upper=0.40 effort=1000.0 velocity=0.1
- added joint stage2_lift_joint: type prismatic, parent stage1_lift_link, child stage2_lift_link, origin xyz=0.19 0 0.423 rpy=0 0 0, axis 0 0 1, limit lower=0.0 upper=1.0 effort=500.0 velocity=0.2
- added joint stage3_horizontal_joint: type prismatic, parent stage2_lift_link, child stage3_horizontal_link, origin xyz=0 0 0.10 rpy=0 0 0, axis 0 1 0, limit lower=-0.196 upper=0.196 effort=500.0 velocity=0.2
- added joint stage4_rotate_joint: type revolute, parent stage3_horizontal_link, child stage4_rotate_link, origin xyz=0.06 0.06 0.0 rpy=1.5708 0 1.5708, axis 0 0 1, limit lower=-3.1416 upper=3.1416 effort=100.0 velocity=1.0
- joint drill_tip_joint: parent gantry_rotate_link -> stage4_rotate_link

File: robo_drill_description/description/robo_drill.urdf.xacro (robot description, xacro)
@@ -16,55 +16,48 @@
     <xacro:include filename="pokeye_base_links.xacro"/>
     <xacro:include filename="sick_multiscan.xacro"/>
-    <xacro:include filename="os-dome.xacro"/>
     <xacro:include filename="realsense_camera.xacro"/>
     <!-- <xacro:include filename="oak_camera.xacro"/> -->
     <!-- Front-right Sick lidar -->
+    <!-- Parented directly to turret_link; origin composed from the previous
+         mount pose so the physical lidar placement is unchanged. -->
     <xacro:sick_multiscan_sensor
-        parent_link="os_sensor_mount"
+        parent_link="turret_link"
         namespace="front"
         sick_link="front_sick_scan"
         sick_scan_link="front_sick"
         sick_imu_link="front_sick_imu"
-        origin_xyz="-0.002 0.243 -0.081"
-        origin_rpy="1.130 0.938 1.453"
+        origin_xyz="0.3535 -0.2430 0.4505"
+        origin_rpy="-0.3457 -0.0696 -2.5121"
     />
     <!-- Sick lidar at back-left of robot -->
+    <!-- Parented directly to turret_link; origin composed from the previous
+         mount pose so the physical lidar placement is unchanged. -->
     <xacro:sick_multiscan_sensor
-        parent_link="os_sensor_mount"
+        parent_link="turret_link"
         namespace="rear"
         sick_link="rear_sick_scan"
         sick_scan_link="rear_sick"
         sick_imu_link="rear_sick_imu"
-        origin_xyz="-0.002 -0.252 -0.788"
-        origin_rpy="-1.98 -0.973 -1.496"
+        origin_xyz="-0.3535 0.2520 0.4505"
+        origin_rpy="-0.3473 -0.0421 0.5965"
     />
-    <!-- Add third sick lidar only in simulation -->
-    <xacro:if value="$(arg simulation)">
-        <xacro:sick_multiscan_sensor
-            parent_link="os_sensor_mount"
-            namespace="dome"
-            sick_link="os_lidar"
-            sick_scan_link="dome_scan"
-            sick_imu_link="dome_imu"
-            origin_xyz="0 0 0"
-            origin_rpy="0 0 0"
-        />
-    </xacro:if>
     <!-- Front RealSense D435i (forward facing) - legacy frames/topics preserved -->
+    <!-- Parented directly to turret_link; origin composed from the previous
+         mount pose so the physical camera placement is unchanged. -->
     <xacro:realsense_d435
-        parent_link="os_sensor_mount"
+        parent_link="turret_link"
         camera_name="camera"
         topic_ns="camera/camera"
-        origin_xyz="0.0075 -0.128 0.015"
-        origin_rpy="-2.998 -1.541 -0.145"
+        origin_xyz="0.4495 0.1280 0.4600"
+        origin_rpy="-0.0015 -0.0295 0.0043"
     />
     <!-- Rear RealSense D435i (back of turret, for localization and mapping) -->
-    <!-- TODO: replace origin with the measured pose of the rear camera on os_sensor_mount -->
+    <!-- TODO: replace origin with the measured pose of the rear camera on turret_link -->
     <xacro:realsense_d435
-        parent_link="os_sensor_mount"
+        parent_link="turret_link"
         camera_name="camera_rear"
         topic_ns="camera_rear"
-        origin_xyz="0.0075 0.128 -0.84"
-        origin_rpy="-0.143 1.541 -0.145"
+        origin_xyz="-0.4055 -0.1280 0.4600"
+        origin_rpy="0.0021 -0.0295 3.1373"
     />
     <xacro:include filename="robodrill_diffdrive_control.xacro" />

File: robo_drill_description/description/robodrill_diffdrive_control.xacro (robot description, xacro)
@@ -65,20 +65,20 @@
             </hardware>
         </xacro:unless>
-        <joint name="gantry_z_joint">
+        <joint name="stage1_lift_joint">
             <command_interface name="position"/>
             <state_interface name="position"/>
             <state_interface name="velocity"/>
         </joint>
-        <joint name="gantry_y_joint">
+        <joint name="stage2_lift_joint">
             <command_interface name="position"/>
             <state_interface name="position"/>
             <state_interface name="velocity"/>
         </joint>
-        <joint name="gantry_x_joint">
+        <joint name="stage3_horizontal_joint">
             <command_interface name="position"/>
             <state_interface name="position"/>
             <state_interface name="velocity"/>
         </joint>
-        <joint name="gantry_rot_joint">
+        <joint name="stage4_rotate_joint">
             <command_interface name="position"/>
             <state_interface name="position"/>

Commit message: Swap stages 3 and 4 to properly represent Pokeye mechanical design.

File: robo_drill_description/description/mobile_manipulator.urdf.xacro (robot description, xacro)
@@ -104,5 +104,5 @@
     />
     <!-- Pokeye has no UR10e manipulator. The 3-stage linear-actuator gantry
-         (stage1_lift_link -> stage2_lift_link -> stage3_horizontal_link -> stage4_rotate_link) is
+         (stage1_lift_link -> stage2_lift_link -> stage3_rotate_link -> stage4_horizontal_link) is
          defined in pokeye_base.urdf and is shared by both robo_drill.urdf.xacro
          and this file. The former UR10e + sensor_plate mount has been removed. -->

File: robo_drill_description/description/pokeye_base.urdf (robot description, URDF)
Before this commit: robot Pokeye, 12 links, 11 joints
Links:
- removed link stage3_horizontal_link
- removed link stage4_rotate_link
- added link stage3_rotate_link, mass 1.0; collision mesh filename=package://robo_drill/robo_drill_description/meshes/d_e_stag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 scale=0.001 0.001 0.001; visual mesh filename=package://robo_drill/robo_drill_description/meshes/d_e_stag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 scale=0.001 0.001 0.001
- added link stage4_horizontal_link, mass 0.5; collision box size=0.08 0.08 0.15
- link stage2_lift_link: geometry collision mesh filename=package://robo_drill/robo_drill_description/meshes/rotatory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 scale=0.001 0.001 0.001; visual mesh filename=package://robo_drill/robo_drill_description/meshes/rotatory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 scale=0.001 0.001 0.001
Joints:
- removed joint stage3_horizontal_joint
- removed joint stage4_rotate_joint
- added joint stage3_rotate_joint: type revolute, parent stage2_lift_link, child stage3_rotate_link, origin xyz=0.08 0 0.10 rpy=1.5708 0 1.5708, axis 0 0 1, limit lower=-3.1416 upper=3.1416 effort=100.0 velocity=1.0
- added joint stage4_horizontal_joint: type prismatic, parent stage3_rotate_link, child stage4_horizontal_link, origin xyz=0.0 0.0 0.08 rpy=-1.5708 -1.5708 0, axis 0 1 0, limit lower=-0.196 upper=0.196 effort=500.0 velocity=0.2
- joint drill_tip_joint: parent stage4_rotate_link -> stage4_horizontal_link
- joint stage2_lift_joint: origin xyz=0.19 0 0.423 rpy=0 0 0 -> xyz=0.15 0 0.423 rpy=0 0 0

File: robo_drill_description/description/robodrill_diffdrive_control.xacro (robot description, xacro)
@@ -75,10 +75,10 @@
             <state_interface name="velocity"/>
         </joint>
-        <joint name="stage3_horizontal_joint">
+        <joint name="stage3_rotate_joint">
             <command_interface name="position"/>
             <state_interface name="position"/>
             <state_interface name="velocity"/>
         </joint>
-        <joint name="stage4_rotate_joint">
+        <joint name="stage4_horizontal_joint">
             <command_interface name="position"/>
             <state_interface name="position"/>
